File: KiCad/Electronics Club/Electronics Club.kicad_pcb (KiCad board)
At the start: 2 copper layers, 60.3 x 80.3 mm, 38 parts, among them J1 Conn_01x05_Female, SW1 Power Switch, U2 LD1117S50TR_SOT223, U3 ATmega328P-AU, Y1 16MHz

Commit message: Generated paste files for stencil
Parts:
- Y1: footprint Crystal:Crystal_SMD_FOX_FQ7050-2Pin_7.0x5.0mm_HandSoldering -> Crystal:Crystal_SMD_7050-2Pin_7.0x5.0mm_HandSoldering
